File: AlveoU25_JTAG_Adapter.kicad_pcb (KiCad board)
At the start: 2 copper layers, 8 parts, among them J1 Xilinx_JTAG, J2 UART, U1 Alveo_U25_Debug

Commit message: PCB Finished - Just JTAG
Parts:
- removed J2: UART, Connector_PinHeader_2.54mm:PinHeader_1x04_P2.54mm_Vertical
- removed R5: 0, Resistor_SMD:R_0603_1608Metric_Pad0.98x0.95mm_HandSolder
- added J3: OTHER, Connector_PinHeader_2.54mm:PinHeader_2x05_P2.54mm_Vertical, F.Cu at (82.6, 56.2)
- added J4: OTHER, Connector_PinHeader_2.54mm:PinHeader_2x06_P2.54mm_Vertical, F.Cu at (85.1, 73.7)
- added R6: 0, Resistor_SMD:R_0603_1608Metric_Pad0.98x0.95mm_HandSolder, B.Cu at (62.8, 65.4)
- added R7: 0, Resistor_SMD:R_0603_1608Metric_Pad0.98x0.95mm_HandSolder, B.Cu at (61.0, 62.1)
- added R8: 0, Resistor_SMD:R_0603_1608Metric_Pad0.98x0.95mm_HandSolder, B.Cu at (59.2, 65.4)
- moved R1 9.79 mm to (88.6, 68.0)
- moved R2 9.79 mm to (88.6, 66.0)
- moved R4 9.79 mm to (88.6, 62.0)
- moved R3 9.79 mm to (88.6, 64.0)
- moved J1 9.71 mm to (95.0, 64.0)
- moved U1 1.50 mm to (61.0, 66.0)
Connections:
- J1 pad 14: HALT -> INIT
- U1 pad A10: unconnected-(U1-PadA10) -> A10
- U1 pad A11: unconnected-(U1-PadA11) -> A11
- U1 pad A12: unconnected-(U1-PadA12) -> A12
- U1 pad A13: unconnected-(U1-PadA13) -> A13
- U1 pad A2: unconnected-(U1-PadA2) -> TCK
- U1 pad A3: unconnected-(U1-PadA3) -> TDI
- U1 pad A4: unconnected-(U1-PadA4) -> TMS
- U1 pad A5: unconnected-(U1-PadA5) -> TDO
- U1 pad A6: unconnected-(U1-PadA6) -> +VREF
- U1 pad A8: unconnected-(U1-PadA8) -> A8
- U1 pad A9: unconnected-(U1-PadA9) -> A9
- U1 pad B10: unconnected-(U1-PadB10) -> B10
- U1 pad B11: unconnected-(U1-PadB11) -> B11
- U1 pad B12: unconnected-(U1-PadB12) -> B12
- U1 pad B13: unconnected-(U1-PadB13) -> B13
- U1 pad B2: unconnected-(U1-PadB2) -> B2
- U1 pad B3: unconnected-(U1-PadB3) -> B3
- U1 pad B4: unconnected-(U1-PadB4) -> B4
- U1 pad B5: unconnected-(U1-PadB5) -> B5
- U1 pad B6: unconnected-(U1-PadB6) -> B6
- U1 pad B8: unconnected-(U1-PadB8) -> B8
- U1 pad B9: unconnected-(U1-PadB9) -> B9
- U1 pad MP: (no net) -> GND
Routing:
- net GND: track 0.00 -> 158.0 mm, vias 0 -> 76
- net +VREF: track 0.00 -> 75.9 mm
- net TDI: track 0.00 -> 40.9 mm, vias 0 -> 2
- net TDO: track 0.00 -> 40.8 mm, vias 0 -> 2
- net TMS: track 0.00 -> 39.5 mm
- net TCK: track 0.00 -> 39.3 mm
- net A9: track 0.00 -> 28.7 mm
- net B9: track 0.00 -> 28.2 mm
- net A8: track 0.00 -> 27.5 mm
- net B13: track 0.00 -> 26.3 mm
- net B11: track 0.00 -> 24.7 mm
- net B8: track 0.00 -> 24.4 mm
- net A10: track 0.00 -> 23.8 mm
- net A11: track 0.00 -> 21.6 mm, vias 0 -> 1
- net B10: track 0.00 -> 21.3 mm
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- added copper zone on B.Cu, net GND
- added copper zone on F.Cu, net GND
Other:
- board outline added: 45 x 31.5 mm

Commit message: Second Revision
Parts:
- removed R8: 0, Resistor_SMD:R_0603_1608Metric_Pad0.98x0.95mm_HandSolder
- added C4: 0u1, Capacitor_SMD:C_0603_1608Metric_Pad1.08x0.95mm_HandSolder, F.Cu at (78.2, 89.9)
- added C5: 0u1, Capacitor_SMD:C_0603_1608Metric_Pad1.08x0.95mm_HandSolder, F.Cu at (74.7, 87.6)
- added J5: Conn_01x06, Connector_PinSocket_2.54mm:PinSocket_1x06_P2.54mm_Vertical, F.Cu at (86.9, 90.2)
- added J6: Conn_02x02_Counter_Clockwise, Connector_PinSocket_2.54mm:PinSocket_2x02_P2.54mm_Vertical, F.Cu at (75.4, 77.5)
- added J7: Conn_01x06, Connector_PinSocket_2.54mm:PinSocket_1x06_P2.54mm_Vertical, F.Cu at (70.4, 90.2)
- added JP1: Conn_01x06, Connector_PinSocket_2.54mm:PinSocket_1x06_P2.54mm_Vertical, F.Cu at (106.0, 87.7)
- added JP2: Conn_01x06, Connector_PinSocket_2.54mm:PinSocket_1x06_P2.54mm_Vertical, F.Cu at (106.0, 77.5)
- added R14: 10k, Resistor_SMD:R_0603_1608Metric_Pad0.98x0.95mm_HandSolder, F.Cu at (81.8, 80.3)
- added R15: 10k, Resistor_SMD:R_0603_1608Metric_Pad0.98x0.95mm_HandSolder, F.Cu at (81.8, 77.2)
- added R9: 0, Resistor_SMD:R_0603_1608Metric_Pad0.98x0.95mm_HandSolder, F.Cu at (74.4, 82.8)
- added U5: 74AVC4T774PW, Package_SO:TSSOP-16_4.4x5mm_P0.65mm, F.Cu at (80.5, 85.1)
- J3: value OTHER -> Conn_02x04_Odd_Even; footprint Connector_PinHeader_2.54mm:PinHeader_2x05_P2.54mm_Vertical -> Connector_PinSocket_2.54mm:PinSocket_2x04_P2.54mm_Vertical
- J4: value OTHER -> Conn_02x04_Odd_Even; footprint Connector_PinHeader_2.54mm:PinHeader_2x06_P2.54mm_Vertical -> Connector_PinSocket_2.54mm:PinSocket_2x04_P2.54mm_Vertical
- moved J3 5.20 mm to (77.5, 57.2)
- moved J4 5.12 mm to (81.3, 70.3)
- moved R1 4.02 mm to (89.0, 64.0)
- moved R2 4.02 mm to (89.0, 62.0)
- moved R3 4.02 mm to (89.0, 60.0)
- moved R4 4.02 mm to (89.0, 58.0)
- moved J1 4.00 mm to (95.0, 60.0)
Connections:
- J3 pad 3: unconnected-(J3-Pad3) -> B6
- J3 pad 5: B6 -> B5
- J3 pad 6: unconnected-(J3-Pad6) -> B4
- J3 pad 7: B4 -> PS_INIT_B
- J3 pad 8: B5 -> PS_POR_B
- J4 pad 1: B8 -> GND
- J4 pad 2: B9 -> nINT
- J4 pad 3: B10 -> MGTAVcc
- J4 pad 4: B11 -> B12
- J4 pad 5: B12 -> B11
- J4 pad 6: B13 -> B10
- J4 pad 7: A8 -> B9
- J4 pad 8: A9 -> SFP_PWR
- U1 pad A10: A10 -> SDA
- U1 pad A11: A11 -> SCL
- U1 pad A12: A12 -> nINT
- U1 pad A13: A13 -> +1V8
- U1 pad A8: A8 -> RXD
- U1 pad A9: A9 -> TXD
- U1 pad B13: B13 -> MGTAVcc
- U1 pad B2: B2 -> PS_POR_B
- U1 pad B3: B3 -> PS_INIT_B
- U1 pad B8: B8 -> SFP_PWR
Routing:
- net GND: track 158.0 -> 406.4 mm, vias 76 -> 126
- net +3V3: track 0.00 -> 56.2 mm, vias 0 -> 2
- net SDA: track 0.00 -> 42.0 mm, vias 0 -> 2
- net SCL: track 0.00 -> 41.9 mm, vias 0 -> 2
- net +1V8: track 0.00 -> 37.8 mm, vias 0 -> 1
- net TXD: track 0.00 -> 34.2 mm
- net RXD: track 0.00 -> 33.8 mm
- net nINT: track 0.00 -> 31.8 mm, vias 0 -> 2
- net A9: track 28.7 -> 0.00 mm
- net MCP2221_TXD: track 0.00 -> 27.5 mm
- net A8: track 27.5 -> 0.00 mm
- net B13: track 26.3 -> 0.00 mm
- net MCP2221_RXD: track 0.00 -> 25.3 mm, vias 0 -> 1
- net B8: track 24.4 -> 0.00 mm
- net A10: track 23.8 -> 0.00 mm
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Other:
- board size 45 x 31.5 mm -> 52.5 x 45.5 mm
- board text added: "Adafruit 4471 MCP2221A"
- board text added: "Alveo U25 Debug Adapter"
